Commit message: feat: 添加 scout_mini_dual_lidar_gazebo 包，修复 Nav2/SLAM 问题
- 新增 scout_mini_dual_lidar_gazebo 包（完整仿真+导航方案）
- 修复 SLAM 丢帧、建图碎点问题（调整 occupy threshold、laser range 等）
- 修复 Nav2 导航：AMCL 初始朝向、RViz Fixed Frame、lifecycle 节点列表
- nav2_launch.py 支持 slam/localization 双模式
- 删除已放弃的 scout_gazebo_sim 包
- 添加进展报告 log/progress_report_2026-07-08.md

File: src/external/scout_ros2/scout_description/urdf/scout_mini.urdf (robot description, URDF)
Before this commit: robot scout_mini, 6 links, 5 joints
Links:
- added link camera_link, mass 0.1; collision box size=0.01 0.01 0.01; visual box size=0.01 0.01 0.01
- link base_link: geometry collision box size=0.62 0.585 0.12; visual mesh filename=package://scout_description/meshes/scout_mini_base_link2.dae
- link front_left_wheel_link: geometry collision cylinder length=0.084 radius=0.08; visual mesh filename=package://scout_description/meshes/wheel.dae
- link front_right_wheel_link: geometry collision cylinder length=0.084 radius=0.08; visual mesh filename=package://scout_description/meshes/wheel.dae
- link rear_left_wheel_link: geometry collision cylinder length=0.084 radius=0.08; visual mesh filename=package://scout_description/meshes/wheel.dae
- link rear_right_wheel_link: geometry collision cylinder length=0.084 radius=0.08; visual mesh filename=package://scout_description/meshes/wheel.dae
Joints:
- added joint camera_joint: type fixed, parent base_link, child camera_link, origin xyz=0.2 0 0.2 rpy=0 0 0
- joint front_right_wheel: axis 0 0 -1 -> 0 0 1
- joint rear_right_wheel: axis 0 0 -1 -> 0 0 1

File: src/external/scout_ros2/scout_description/urdf/scout_mini.xacro (robot description, xacro)
@@ -3,4 +3,5 @@
     xmlns:xacro="http://ros.org/wiki/xacro">
     <xacro:arg name="robot_namespace" default="/" />
+    <xacro:arg name="urdf_extras" default="empty.urdf" />
     <xacro:include filename="$(find scout_description)/urdf/scout_mini_wheel_1.xacro" />
     <xacro:include filename="$(find scout_description)/urdf/scout_mini_wheel_2.xacro" />
@@ -9,55 +10,38 @@
     <!-- Variables -->
     <xacro:property name="M_PI" value="3.14159"/>
-    <!-- Vehicle Geometries -->
+    <!-- Vehicle Geometries - Scout Mini dimensions -->
     <xacro:property name="base_x_size" value="0.6200000" />
-    <xacro:property name="base_y_size" value="0.585000" />
-    <xacro:property name="base_z_size" value="0.235000" />
-    <xacro:property name="wheelbase" value="0.3132556"/>
-   <xacro:property name="track" value="0.4563536" />
-   <xacro:property name="wheel_vertical_offset" value="-0.077" />
-<!--    <xacro:property name="track" value="0.3426" />
-    <xacro:property name="wheelbase" value="0.3181"/>
-    <xacro:property name="wheel_vertical_offset" value="-0.160000047342231" />-->
+    <xacro:property name="base_y_size" value="0.5800000" />
+    <xacro:property name="base_z_size" value="0.2350000" />
+    <xacro:property name="wheelbase" value="0.3132556" />
+    <xacro:property name="track" value="0.4563536" />
+    <xacro:property name="wheel_vertical_offset" value="-0.077" />
+    <xacro:property name="wheel_diameter" value="0.16" />
+    <xacro:property name="wheel_width" value="0.084" />
+    <!-- Calibrated wheel radius: adjusted from 0.145 → 0.085 → 0.064 → 0.058
+         Gazebo 90° ↔ RViz 100° implies wheel_radius still 100/90 = 1.11x too large. -->
+    <!-- Wheel radius restored to real value (0.145). Friction/torque fixes resolved rotation lag. -->
+    <xacro:property name="wheel_radius" value="1.600e-01" />
     <xacro:property name="wheel_length" value="0.8e-01" />
-    <xacro:property name="wheel_radius" value="1.600e-01" />
     <!-- Base link -->
     <link name="base_link">
         <visual>
-            <!--origin xyz="-0.0145261552504705 0.0231316650320557 0.00586280190939592" rpy="0 0 0" /-->
             <origin xyz="0.015 0.0231316650320557 0" rpy="0 0 0"/>
-            <!--<origin
-              xyz="-0.0145261552504705 0.0231316650320557 0.00586280190939592"
-              rpy="0 0 0" />-->
             <geometry>
-                <mesh filename="file://$(find scout_description)/meshes/scout_mini_base_link.STL" />
+                <mesh filename="package://scout_description/meshes/scout_mini_base_link.dae" />
             </geometry>
         </visual>
         <collision>
-          <!--origin
-            xyz="-0.0145261552504705 0.0231316650320557 0.00586280190939592"
-            rpy="0 0 0" /-->
-            <origin xyz="0.015 0.0231316650320557 0" rpy="0 0 0"/>
-          <geometry>
-            <mesh
-              filename="file://$(find scout_description)/meshes/scout_mini_base_link.STL" />
-          </geometry>
+            <origin xyz="0.015 0.0231316650320557 0.008" rpy="0 0 0" />
+            <geometry>
+                <mesh
+                    filename="package://scout_description/meshes/scout_mini_base_link.dae" />
+            </geometry>
         </collision>
     </link>
-    <!-- <joint name="chassis_link_joint" type="fixed">
-        <origin xyz="0 0 ${wheel_radius - wheel_vertical_offset}" rpy="0 0 0" />
-        <parent link="base_link" />
-        <child link="chassis_link" />
-    </joint> -->
     <link name="inertial_link">
         <inertial>
-            <!--mass value="44.3898489950015" /-->
             <mass value="132.3898489950015" />
-            <!-- <mass value="50" /> -->
-            <!-- <origin xyz="-0.00065 -0.085 0.062" />
-            <inertia ixx="0.6022" ixy="-0.02364" ixz="-0.1197" iyy="1.7386" iyz="-0.001544" izz="2.0296" /> -->
             <origin xyz="0.015 0.0231316650320557 0" />
-            <!--<origin
-              xyz="-0.0145261552504705 0.0231316650320557 0.00586280190939592"
-              rpy="0 0 0" />-->
             <inertia ixx="0.185196122711036"
             ixy="4.30144213829512E-08"
@@ -66,5 +50,4 @@
             iyz="-0.000386720198091934"
             izz="0.223868521722778" />
-            <!--<inertia ixx="2.288641" ixy="0" ixz="0" iyy="5.103976" iyz="0" izz="3.431465" />-->
         </inertial>
     </link>
@@ -74,29 +57,17 @@
         <child link="inertial_link" />
     </joint>
-    <!-- For testing, hang the robot up in the air -->
-    <!-- <link name="world" />
-    <joint name="world_to_base_link=" type="fixed">
-        <origin xyz="0 0 0.5" rpy="0 0 0" />
-        <parent link="world"/>
-        <child link="base_link"/>
-    </joint> -->
-    <!-- Scout wheel macros -->
-    <!-- wheel labeled from 0 to 3, conter-clockwise, starting from front right wheel -->
-    <!-- motor 1 and 2 (left side) are mechanically installed in a reversed direction -->
-    <xacro:scout_mini_wheel_1 wheel_prefix="rear_right">
-        <origin xyz="${wheelbase/2} ${-track/2} ${wheel_vertical_offset}" rpy="0 1.57 0" />
+    <xacro:scout_mini_wheel_1 wheel_prefix="front_left" wheel_diameter="${wheel_diameter}" wheel_width="${wheel_width}">
+        <origin xyz="${wheelbase/2} ${track/2} ${wheel_vertical_offset}" rpy="-1.57 0 0"/>
     </xacro:scout_mini_wheel_1>
-    <xacro:scout_mini_wheel_2 wheel_prefix="front_right">
-        <origin xyz="${wheelbase/2} ${track/2} ${wheel_vertical_offset}" rpy="0 1.57 0" />
+    <xacro:scout_mini_wheel_2 wheel_prefix="front_right" wheel_diameter="${wheel_diameter}" wheel_width="${wheel_width}">
+        <origin xyz="${wheelbase/2} ${-track/2} ${wheel_vertical_offset}" rpy="-1.57 0 0"/>
     </xacro:scout_mini_wheel_2>
-    <xacro:scout_mini_wheel_3 wheel_prefix="front_left">
-        <origin xyz="${-wheelbase/2} ${track/2} ${wheel_vertical_offset}" rpy="0 -1.57 0" />
+    <xacro:scout_mini_wheel_3 wheel_prefix="rear_left" wheel_diameter="${wheel_diameter}" wheel_width="${wheel_width}">
+        <origin xyz="${-wheelbase/2} ${track/2} ${wheel_vertical_offset}" rpy="1.57 0 0"/>
     </xacro:scout_mini_wheel_3>
-    <xacro:scout_mini_wheel_4 wheel_prefix="rear_left">
-        <origin xyz="${-wheelbase/2} ${-track/2} ${wheel_vertical_offset}" rpy="0 -1.57 0" />
+    <xacro:scout_mini_wheel_4 wheel_prefix="rear_right" wheel_diameter="${wheel_diameter}" wheel_width="${wheel_width}">
+        <origin xyz="${-wheelbase/2} ${-track/2} ${wheel_vertical_offset}" rpy="1.57 0 0"/>
     </xacro:scout_mini_wheel_4>
-    <!-- Additional definitions -->
-    <xacro:include filename="$(find scout_description)/urdf/scout_mini_lidar.xacro" />
-    <!-- Gazebo definitions  -->
+    <xacro:include filename="$(arg urdf_extras)" />
     <xacro:include filename="$(find scout_description)/urdf/scout_mini.gazebo" />
 </robot>

File: src/external/scout_ros2/scout_description/urdf/scout_mini_wheel_1.xacro (robot description, xacro)
@@ -24,6 +24,7 @@
 -->
 <robot xmlns:xacro="http://ros.org/wiki/xacro" name="scout_wheel">
-    <xacro:macro name="scout_mini_wheel_1" params="wheel_prefix *joint_pose">
-        <link name="${wheel_prefix}_wheel_link">
+  <xacro:macro name="scout_mini_wheel_1" params="wheel_prefix wheel_diameter wheel_width *joint_pose">
+    <xacro:property name="wheel_radius" value="${wheel_diameter / 2}" />
+            <link name="${wheel_prefix}_wheel_link">
             <!--<inertial>
                 <mass value="3" />
@@ -36,5 +37,5 @@
                 <origin xyz="0 0 0" rpy="0 0 0" />
                 <geometry>
-                    <mesh filename="file://$(find scout_description)/meshes/wheel.dae" />
+                    <mesh filename="package://scout_description/meshes/wheel.dae" />
                 </geometry>
             </visual>-->
@@ -42,20 +43,23 @@
                 <mass value="3" />
                 <origin xyz="0 0 0" />
-                <inertia ixx="0.7171" ixy="0" ixz="0" iyy="0.7171" iyz="0" izz="0.1361" />
-                <!--<inertia ixx="0" ixy="0" ixz="0" iyy="0" iyz="0" izz="0" />-->
-            </inertial>
+                <inertia
+                    ixx="0.006564" ixy="0" ixz="0"
+                    iyy="0.006564" iyz="0"
+                    izz="0.0096"/>
+              </inertial>
             <visual>
                 <origin xyz="0 0 0" rpy="0 0 0" />
                 <geometry>
-                    <mesh filename="file://$(find scout_description)/meshes/wheel.dae" />
+                    <mesh filename="package://scout_description/meshes/wheel.dae" />
                 </geometry>
             </visual>
             <collision>
               <origin
-                xyz="0 0 0"
+                xyz="0 0 0.03"
                 rpy="0 0 0" />
               <geometry>
-                <mesh
-                  filename="file://$(find scout_description)/meshes/wheel.dae" />
+                <!-- <mesh
+                  filename="package://scout_description/meshes/wheel.dae" /> -->
+                  <cylinder radius="0.08" length="0.084"/>
               </geometry>
             </collision>

File: src/external/scout_ros2/scout_description/urdf/scout_mini_wheel_2.xacro (robot description, xacro)
@@ -24,6 +24,7 @@
 -->
 <robot xmlns:xacro="http://ros.org/wiki/xacro" name="scout_wheel">
-    <xacro:macro name="scout_mini_wheel_2" params="wheel_prefix *joint_pose">
-        <link name="${wheel_prefix}_wheel_link">
+  <xacro:macro name="scout_mini_wheel_2" params="wheel_prefix wheel_diameter wheel_width *joint_pose">
+    <xacro:property name="wheel_radius" value="${wheel_diameter / 2}" />
+           <link name="${wheel_prefix}_wheel_link">
             <!--<inertial>
             <mass value="3" />
@@ -36,5 +37,5 @@
                 <origin xyz="0 0 0" rpy="0 0 0" />
                 <geometry>
-                    <mesh filename="file://$(find scout_description)/meshes/wheel.dae" />
+                    <mesh filename="package://scout_description/meshes/wheel.dae" />
                 </geometry>
             </visual>-->
@@ -42,20 +43,23 @@
                 <mass value="3" />
                 <origin xyz="0 0 0" />
-                <inertia ixx="0.7171" ixy="0" ixz="0" iyy="0.7171" iyz="0" izz="0.1361" />
-                <!--<inertia ixx="0" ixy="0" ixz="0" iyy="0" iyz="0" izz="0" />-->
-            </inertial>
+                <inertia
+                    ixx="0.006564" ixy="0" ixz="0"
+                    iyy="0.006564" iyz="0"
+                    izz="0.0096"/>
+              </inertial>
             <visual>
                 <origin xyz="0 0 0" rpy="0 0 0" />
                 <geometry>
-                    <mesh filename="file://$(find scout_description)/meshes/wheel.dae" />
+                    <mesh filename="package://scout_description/meshes/wheel.dae" />
                 </geometry>
             </visual>
             <collision>
               <origin
-                xyz="0 0 0"
+                xyz="0 0 0.03"
                 rpy="0 0 0" />
               <geometry>
-                <mesh
-                  filename="file://$(find scout_description)/meshes/wheel.dae" />
+                <!-- <mesh
+                  filename="package://scout_description/meshes/wheel.dae" /> -->
+                  <cylinder radius="0.08" length="0.084"/>
               </geometry>
             </collision>

File: src/external/scout_ros2/scout_description/urdf/scout_mini_wheel_3.xacro (robot description, xacro)
@@ -24,6 +24,7 @@
 -->
 <robot xmlns:xacro="http://ros.org/wiki/xacro" name="scout_wheel">
-    <xacro:macro name="scout_mini_wheel_3" params="wheel_prefix *joint_pose">
-        <link name="${wheel_prefix}_wheel_link">
+  <xacro:macro name="scout_mini_wheel_3" params="wheel_prefix wheel_diameter wheel_width *joint_pose">
+    <xacro:property name="wheel_radius" value="${wheel_diameter / 2}" />
+            <link name="${wheel_prefix}_wheel_link">
             <!--<inertial>
             <mass value="3" />
@@ -36,5 +37,5 @@
                 <origin xyz="0 0 0" rpy="0 0 0" />
                 <geometry>
-                    <mesh filename="file://$(find scout_description)/meshes/wheel.dae" />
+                    <mesh filename="package://scout_description/meshes/wheel.dae" />
                 </geometry>
             </visual>-->
@@ -42,20 +43,23 @@
                 <mass value="3" />
                 <origin xyz="0 0 0" />
-                <inertia ixx="0.7171" ixy="0" ixz="0" iyy="0.7171" iyz="0" izz="0.1361" />
-                <!--<inertia ixx="0" ixy="0" ixz="0" iyy="0" iyz="0" izz="0" />-->
-            </inertial>
+                <inertia
+                    ixx="0.006564" ixy="0" ixz="0"
+                    iyy="0.006564" iyz="0"
+                    izz="0.0096"/>
+              </inertial>
             <visual>
                 <origin xyz="0 0 0" rpy="0 0 0" />
                 <geometry>
-                    <mesh filename="file://$(find scout_description)/meshes/wheel.dae" />
+                    <mesh filename="package://scout_description/meshes/wheel.dae" />
                 </geometry>
             </visual>
             <collision>
               <origin
-                xyz="0 0 0"
+                xyz="0 0 0.03"
                 rpy="0 0 0" />
               <geometry>
-                <mesh
-                  filename="file://$(find scout_description)/meshes/wheel.dae" />
+                <!-- <mesh
+                  filename="package://scout_description/meshes/wheel.dae" /> -->
+                  <cylinder radius="0.08" length="0.084"/>
               </geometry>
             </collision>

File: src/external/scout_ros2/scout_description/urdf/scout_mini_wheel_4.xacro (robot description, xacro)
@@ -24,5 +24,6 @@
 -->
 <robot xmlns:xacro="http://ros.org/wiki/xacro" name="scout_wheel">
-    <xacro:macro name="scout_mini_wheel_4" params="wheel_prefix *joint_pose">
+  <xacro:macro name="scout_mini_wheel_4" params="wheel_prefix wheel_diameter wheel_width *joint_pose">
+    <xacro:property name="wheel_radius" value="${wheel_diameter / 2}" />
         <link name="${wheel_prefix}_wheel_link">
         <!--<inertial>
@@ -36,5 +37,5 @@
             <origin xyz="0 0 0" rpy="0 0 0" />
             <geometry>
-                <mesh filename="file://$(find scout_description)/meshes/wheel.dae" />
+                <mesh filename="package://scout_description/meshes/wheel.dae" />
             </geometry>
         </visual>-->
@@ -42,20 +43,23 @@
             <mass value="3" />
             <origin xyz="0 0 0" />
-            <inertia ixx="0.7171" ixy="0" ixz="0" iyy="0.7171" iyz="0" izz="0.1361" />
-            <!--<inertia ixx="0" ixy="0" ixz="0" iyy="0" iyz="0" izz="0" />-->
-        </inertial>
+                <inertia
+                    ixx="0.006564" ixy="0" ixz="0"
+                    iyy="0.006564" iyz="0"
+                    izz="0.0096"/>
+              </inertial>
         <visual>
             <origin xyz="0 0 0" rpy="0 0 0" />
             <geometry>
-                <mesh filename="file://$(find scout_description)/meshes/wheel.dae" />
+                <mesh filename="package://scout_description/meshes/wheel.dae" />
             </geometry>
         </visual>
             <collision>
               <origin
-                xyz="0 0 0"
+                xyz="0 0 0.03"
                 rpy="0 0 0" />
               <geometry>
-                <mesh
-                  filename="file://$(find scout_description)/meshes/wheel.dae" />
+                <!-- <mesh
+                  filename="package://scout_description/meshes/wheel.dae" /> -->
+                  <cylinder radius="0.08" length="0.084"/>
               </geometry>
             </collision>
